File: hardware/BzBrd_1_0_0.brd (EAGLE design)
At the start: 88.9 x 38.1 mm, 48 parts, among them J1 5.5x2.1mm Barrel, U1 BQ24075, U2 BQ27441-G1, U3 SHT31-DIS, U4 OPA344, U5 AKU342-, U7 MMA8452Q

Commit message: one schematic sheet
Parts:
- added FRAME1: FRAME-LEDGER, SparkFun-Aesthetics:CREATIVE_COMMONS
Changed lines of the file:
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@@
 <attribute name="SF_ID" value="PRT-12748" x="83.82" y="13.97" size="1.778" layer="27" rot="R180" display="off"/>
 </element>
+<element name="FRAME1" library="SparkFun-Aesthetics" package="CREATIVE_COMMONS" value="FRAME-LEDGER" x="-87.63" y="-8.89"/>
 </elements>
 <signals>
