File: hardware/BzBrd_1_0_0.sch (EAGLE design)
At the start: 44 parts, among them J1 5.5x2.1mm Barrel, U1 BQ24075, U2 BQ27441-G1, U3 SHT31-DIS, U4 OPA344, U5 AKU342-, U7 MMA8452Q

Commit message: one schematic sheet
Parts:
- added FRAME1: FRAME-LEDGER, SparkFun-Aesthetics:FRAME-LEDGER
Other:
- note added: "MMA8452 accelerometer"
- note added: "Mic and Pre-Amp"
- note added: "MicroSD Socket"
- note added: "Photon SoC"
- note added: "SHT30 t/rh"
- note added: "Sets fast charge current - R_ISET range: 590-8.9k - I_CHG = ~885 / R_ISET - EX: R_ISET = 1780 : I_CHG = 0.5A"
- note added: "v1.0.1"
- note removed: "* Add decoupling cap - AD suggests 10uF and 0.1uF after upto 100Ohm resistance"
- note removed: "* Non-cantilevered - added standoffs for stability"
- note removed: "ADMP401 MEMS Microphone + Amp"
- note removed: "I2C Mode"
- note removed: "Jim Lindblom"
- note removed: "Jim Lindblom Mod: Peter Naylor"
- note removed: "Revised by: Patrick Alberts"
- note removed: "SHT31 Environment Sensor"
- note removed: "SJ2: Cut to enable charge timer."
- note removed: "SJ3: Cut to set custom ISET."
- note removed: "SJ4: Cut to set custom ILIM."
- note removed: "SJ5 sets the operation of the power LED. To either: - Power OUT indicator - !PGOOD! indicator (Good IN supply) - Open (LED disconnected)"
- note removed: "Sets fast charge current - R_ISET range: 590-8.9k - I_CHG = ~885 / R_ISET - EX: R_ISET = 590 : I_CHG = 1.5A"
- note removed: "Updates:"
- note removed: "microSD Breakout Board"
- note removed: "v01"
- note removed: "v10"
- note removed: "v14"
